File: led-tester.kicad_pcb (KiCad board)
At the start: 2 copper layers, 50 x 50 mm, 30 parts, among them J1 PWR, J2 PWR, J3 VOLT, J4 LED, SW1 LED_POL, SW2 1mA, SW3 2mA, SW4 3mA, SW5 5mA, SW6 10mA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

Commit message: Final tweaks and some part numbers
Parts:
- L1: value L_Small -> 4u7; footprint Inductor_SMD:L_2512_6332Metric -> Inductor_SMD:L_1008_2520Metric
- SW1: footprint led-tester:MFS201N－4－Z -> led-tester:OS202011MS2QS1
- moved R1 20.9 mm to (120.0, 96.0), turned to -90 degrees
- moved R6 20.9 mm to (130.0, 96.0), turned to -90 degrees
- moved R2 17.1 mm to (122.0, 96.0), turned to -90 degrees
- moved R5 17.1 mm to (128.0, 96.0), turned to -90 degrees
- moved R3 14.8 mm to (124.0, 96.0), turned to -90 degrees
- moved R4 14.8 mm to (126.0, 96.0), turned to -90 degrees
- moved C2 6.42 mm to (117.3, 73.5), turned to -90 degrees
- moved C1 5.28 mm to (114.3, 79.1)
- moved U1 5.28 mm to (114.3, 76.0)
- moved L1 3.38 mm to (114.3, 72.5)
- moved R10 2.77 mm to (133.2, 72.0)
- moved R7 2.77 mm to (133.2, 73.5)
- moved R8 2.77 mm to (133.2, 78.5)
- moved R9 2.77 mm to (137.2, 78.5)
- moved U2 2.77 mm to (135.2, 76.0)
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Connections:
- R1 pad 1: LED- -> Net-(R1-Pad1)
- R1 pad 2: Net-(R1-Pad2) -> GND
- R2 pad 1: LED- -> Net-(R2-Pad1)
- R2 pad 2: Net-(R2-Pad2) -> GND
- R3 pad 1: LED- -> Net-(R3-Pad1)
- R3 pad 2: Net-(R3-Pad2) -> GND
- R4 pad 1: LED- -> Net-(SW5-Pad2)
- R4 pad 2: Net-(R4-Pad2) -> GND
- R5 pad 1: LED- -> Net-(SW6-Pad2)
- R5 pad 2: Net-(R5-Pad2) -> GND
- R6 pad 1: LED- -> Net-(SW7-Pad2)
- R6 pad 2: Net-(R6-Pad2) -> GND
- SW2 pad 1: Net-(R1-Pad2) -> LED-
- SW2 pad 2: GND -> Net-(R1-Pad1)
- SW3 pad 1: Net-(R2-Pad2) -> LED-
- SW3 pad 2: GND -> Net-(R2-Pad1)
- SW4 pad 1: Net-(R3-Pad2) -> LED-
- SW4 pad 2: GND -> Net-(R3-Pad1)
- SW5 pad 1: Net-(R4-Pad2) -> LED-
- SW5 pad 2: GND -> Net-(SW5-Pad2)
- SW6 pad 1: Net-(R5-Pad2) -> LED-
- SW6 pad 2: GND -> Net-(SW6-Pad2)
- SW7 pad 1: Net-(R6-Pad2) -> LED-
- SW7 pad 2: GND -> Net-(SW7-Pad2)
Routing:
- net +5V: track 71.4 -> 0.00 mm
- net LED-: track 65.9 -> 112.8 mm
- net Net-(SW7-Pad2): track 0.00 -> 26.9 mm
- net Net-(R1-Pad1): track 0.00 -> 23.0 mm
- net Net-(SW6-Pad2): track 0.00 -> 20.8 mm
- net Net-(R2-Pad1): track 0.00 -> 17.6 mm
- net Net-(SW5-Pad2): track 0.00 -> 16.1 mm
- net Net-(R3-Pad1): track 0.00 -> 11.7 mm
- net GND: track 6.51 -> 16.6 mm, vias 6 -> 12
- net Net-(R6-Pad2): track 9.88 -> 0.00 mm
- net Net-(R5-Pad2): track 9.88 -> 0.00 mm
- net Net-(R4-Pad2): track 9.88 -> 0.00 mm
- net Net-(R3-Pad2): track 9.88 -> 0.00 mm
- net Net-(R2-Pad2): track 9.88 -> 0.00 mm
- net Net-(R1-Pad2): track 9.88 -> 0.00 mm
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- added copper zone on F.Cu, net +5V
Other:
- outline, holes or cut-outs redrawn

Commit message: Final tweaks and bom
Changed lines of the file:
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@@
   (net 14 "Net-(R2-Pad1)")
   (net 15 "Net-(R3-Pad1)")
-  (net 16 "Net-(SW5-Pad2)")
-  (net 17 "Net-(SW6-Pad2)")
-  (net 18 "Net-(SW7-Pad2)")
+  (net 16 "Net-(R4-Pad1)")
+  (net 17 "Net-(R5-Pad1)")
+  (net 18 "Net-(R6-Pad1)")
   (net 19 "Net-(J4-Pad1)")
   (net 20 "Net-(J4-Pad10)")
@@
       (net 6 "LED-") (pinfunction "1") (pintype "passive"))
     (pad "2" thru_hole circle (at 6.5 4.5 180) (size 2 2) (drill 1.1) (layers *.Cu *.Mask)
-      (net 16 "Net-(SW5-Pad2)") (pinfunction "2") (pintype "passive"))
+      (net 16 "Net-(R4-Pad1)") (pinfunction "2") (pintype "passive"))
     (pad "2" thru_hole circle (at 0 4.5 180) (size 2 2) (drill 1.1) (layers *.Cu *.Mask)
-      (net 16 "Net-(SW5-Pad2)") (pinfunction "2") (pintype "passive"))
+      (net 16 "Net-(R4-Pad1)") (pinfunction "2") (pintype "passive"))
     (model "${KICAD6_3DMODEL_DIR}/Button_Switch_THT.3dshapes/SW_PUSH_6mm_H8mm.wrl"
       (offset (xyz 0 0 0))
@@
       (net 6 "LED-") (pinfunction "1") (pintype "passive"))
     (pad "2" thru_hole circle (at 6.5 4.5 180) (size 2 2) (drill 1.1) (layers *.Cu *.Mask)
-      (net 17 "Net-(SW6-Pad2)") (pinfunction "2") (pintype "passive"))
+      (net 17 "Net-(R5-Pad1)") (pinfunction "2") (pintype "passive"))
     (pad "2" thru_hole circle (at 0 4.5 180) (size 2 2) (drill 1.1) (layers *.Cu *.Mask)
-      (net 17 "Net-(SW6-Pad2)") (pinfunction "2") (pintype "passive"))
+      (net 17 "Net-(R5-Pad1)") (pinfunction "2") (pintype "passive"))
     (model "${KICAD6_3DMODEL_DIR}/Button_Switch_THT.3dshapes/SW_PUSH_6mm_H8mm.wrl"
       (offset (xyz 0 0 0))
@@
     (fp_line (start 0.8 0.4125) (end -0.8 0.4125) (layer "F.Fab") (width 0.1))
     (pad "1" smd roundrect (at -0.825 0 270) (size 0.8 0.95) (layers "F.Cu" "F.Paste" "F.Mask") (roundrect_rratio 0.25)
-      (net 18 "Net-(SW7-Pad2)") (pintype "passive"))
+      (net 18 "Net-(R6-Pad1)") (pintype "passive"))
     (pad "2" smd roundrect (at 0.825 0 270) (size 0.8 0.95) (layers "F.Cu" "F.Paste" "F.Mask") (roundrect_rratio 0.25)
       (net 2 "GND") (pintype "passive"))
@@
     (fp_line (start -0.8 0.4125) (end -0.8 -0.4125) (layer "F.Fab") (width 0.1))
     (pad "1" smd roundrect (at -0.825 0 270) (size 0.8 0.95) (layers "F.Cu" "F.Paste" "F.Mask") (roundrect_rratio 0.25)
-      (net 17 "Net-(SW6-Pad2)") (pintype "passive"))
+      (net 17 "Net-(R5-Pad1)") (pintype "passive"))
     (pad "2" smd roundrect (at 0.825 0 270) (size 0.8 0.95) (layers "F.Cu" "F.Paste" "F.Mask") (roundrect_rratio 0.25)
       (net 2 "GND") (pintype "passive"))
@@
       (net 6 "LED-") (pinfunction "1") (pintype "passive"))
     (pad "2" thru_hole circle (at 0 4.5 180) (size 2 2) (drill 1.1) (layers *.Cu *.Mask)
-      (net 18 "Net-(SW7-Pad2)") (pinfunction "2") (pintype "passive"))
+      (net 18 "Net-(R6-Pad1)") (pinfunction "2") (pintype "passive"))
     (pad "2" thru_hole circle (at 6.5 4.5 180) (size 2 2) (drill 1.1) (layers *.Cu *.Mask)
-      (net 18 "Net-(SW7-Pad2)") (pinfunction "2") (pintype "passive"))
+      (net 18 "Net-(R6-Pad1)") (pinfunction "2") (pintype "passive"))
     (model "${KICAD6_3DMODEL_DIR}/Button_Switch_THT.3dshapes/SW_PUSH_6mm_H8mm.wrl"
       (offset (xyz 0 0 0))
@@
     (fp_line (start -0.8 0.4125) (end -0.8 -0.4125) (layer "F.Fab") (width 0.1))
     (pad "1" smd roundrect (at -0.825 0 270) (size 0.8 0.95) (layers "F.Cu" "F.Paste" "F.Mask") (roundrect_rratio 0.25)
-      (net 16 "Net-(SW5-Pad2)") (pintype "passive"))
+      (net 16 "Net-(R4-Pad1)") (pintype "passive"))
     (pad "2" smd roundrect (at 0.825 0 270) (size 0.8 0.95) (layers "F.Cu" "F.Paste" "F.Mask") (roundrect_rratio 0.25)
       (net 2 "GND") (pintype "passive"))
@@
   (segment (start 115.75 92) (end 115.25 91.5) (width 0.5) (layer "F.Cu") (net 14))
   (segment (start 123.25 83.75) (end 123.25 90.25) (width 0.5) (layer "F.Cu") (net 15))
-  (segment (start 124 92.5) (end 124 95.175) (width 0.5) (layer "F.Cu") (net 15))
-  (segment (start 123.25 91.75) (end 124 92.5) (width 0.5) (layer "F.Cu") (net 15))
-  (segment (start 123.25 90.25) (end 123.25 91.75) (width 0.5) (layer "F.Cu") (net 15))
+  (segment (start 123.25 91.5) (end 124 92.25) (width 0.5) (layer "F.Cu") (net 15))
+  (segment (start 124 92.25) (end 124 95.175) (width 0.5) (layer "F.Cu") (net 15))
+  (segment (start 123.25 90.25) (end 123.25 91.5) (width 0.5) (layer "F.Cu") (net 15))
   (segment (start 130.75 92) (end 126.5 92) (width 0.5) (layer "F.Cu") (net 16))
   (segment (start 131.25 83.75) (end 131.25 90.25) (width 0.5) (layer "F.Cu") (net 16))
