File: led-tester.kicad_sch (KiCad schematic)
At the start: 30 parts, among them J1 PWR, J2 PWR, J3 VOLT, J4 LED, SW1 LED_POL, SW2 1mA, SW3 2mA, SW4 3mA, SW5 5mA, SW6 10mA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

Commit message: Final tweaks and some part numbers
Parts:
- L1: value L_Small -> 4u7; footprint Inductor_SMD:L_2512_6332Metric -> Inductor_SMD:L_1008_2520Metric; LCSC (none) -> C91237
- SW1: footprint led-tester:MFS201N－4－Z -> led-tester:OS202011MS2QS1; Farnell 2854847 -> (none)
- U2: LCSC (none) -> C395460
Connections:
- net GND: now also R1.2, R2.2, R3.2, R4.2, R5.2, R6.2; no longer SW2.2, SW3.2, SW4.2, SW5.2, SW6.2, SW7.2
- net LED-: now also SW2.1, SW3.1, SW4.1, SW5.1, SW6.1, SW7.1; no longer R1.1, R2.1, R3.1, R4.1, R5.1, R6.1
- new net: R6.1, SW7.2
- new net: R1.1, SW2.2
- new net: R3.1, SW4.2
- new net: R4.1, SW5.2
- new net: R2.1, SW3.2
- new net: R5.1, SW6.2
Other:
- moved on the sheet: R1, R2, R3, R4, R5, R6, SW2, SW3, SW4, SW5, SW6, SW7

Commit message: LCSC Part Numbers and BOM
Parts:
- C1, C2: LCSC (none) -> C1713
- J4: LCSC (none) -> 2xC718240
- R1: LCSC (none) -> C105588
- R2: LCSC (none) -> C2759402
- R3: LCSC (none) -> C108661
- R4: LCSC (none) -> C22950
- R5: LCSC (none) -> C109318
- R6: LCSC (none) -> C25197
- SW2, SW3, SW4, SW5, SW6, SW7: LCSC (none) -> C2834903
Changed lines of the file:
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@@
       (effects (font (size 1.27 1.27)) hide)
     )
-    (property "LCSC" "" (id 4) (at 85.09 101.6 0)
+    (property "LCSC" "C2834903" (id 4) (at 85.09 101.6 0)
       (effects (font (size 1.27 1.27)) hide)
     )
@@
       (effects (font (size 1.27 1.27)) hide)
     )
-    (property "LCSC" "" (id 4) (at 85.09 57.15 0)
+    (property "LCSC" "C2834903" (id 4) (at 85.09 57.15 0)
       (effects (font (size 1.27 1.27)) hide)
     )
@@
       (effects (font (size 1.27 1.27)) hide)
     )
-    (property "LCSC" "" (id 4) (at 85.09 74.93 0)
+    (property "LCSC" "C2834903" (id 4) (at 85.09 74.93 0)
       (effects (font (size 1.27 1.27)) hide)
     )
@@
       (effects (font (size 1.27 1.27)) hide)
     )
-    (property "LCSC" "" (id 4) (at 85.09 83.82 0)
+    (property "LCSC" "C2834903" (id 4) (at 85.09 83.82 0)
       (effects (font (size 1.27 1.27)) hide)
     )
@@
       (effects (font (size 1.27 1.27)) hide)
     )
+    (property "LCSC" "C105588" (id 4) (at 92.71 57.15 0)
+      (effects (font (size 1.27 1.27)) hide)
+    )
     (pin "1")
     (pin "2")
@@
       (effects (font (size 1.27 1.27)) hide)
     )
+    (property "LCSC" "C25197" (id 4) (at 92.71 101.6 0)
+      (effects (font (size 1.27 1.27)) hide)
+    )
     (pin "1")
     (pin "2")
@@
     )
     (property "Datasheet" "~" (id 3) (at 120.65 41.91 0)
+      (effects (font (size 1.27 1.27)) hide)
+    )
+    (property "LCSC" "2xC718240" (id 4) (at 120.65 41.91 0)
       (effects (font (size 1.27 1.27)) hide)
     )
@@
       (effects (font (size 1.27 1.27)) hide)
     )
-    (property "LCSC" "" (id 4) (at 85.09 66.04 0)
+    (property "LCSC" "C2834903" (id 4) (at 85.09 66.04 0)
       (effects (font (size 1.27 1.27)) hide)
     )
@@
       (effects (font (size 1.27 1.27)) hide)
     )
-    (property "LCSC" "" (id 4) (at 85.09 92.71 0)
+    (property "LCSC" "C2834903" (id 4) (at 85.09 92.71 0)
       (effects (font (size 1.27 1.27)) hide)
     )
@@
     )
     (property "Datasheet" "~" (id 3) (at 92.71 66.04 0)
+      (effects (font (size 1.27 1.27)) hide)
+    )
+    (property "LCSC" "C2759402" (id 4) (at 92.71 66.04 0)
       (effects (font (size 1.27 1.27)) hide)
     )
@@
       (effects (font (size 1.27 1.27)) hide)
     )
+    (property "LCSC" "C1713" (id 4) (at 88.9 40.64 0)
+      (effects (font (size 1.27 1.27)) hide)
+    )
     (pin "1")
     (pin "2")
@@
       (effects (font (size 1.27 1.27)) hide)
     )
+    (property "LCSC" "C109318" (id 4) (at 92.71 92.71 0)
+      (effects (font (size 1.27 1.27)) hide)
+    )
     (pin "1")
     (pin "2")
@@
       (effects (font (size 1.27 1.27)) hide)
     )
+    (property "LCSC" "C22950" (id 4) (at 92.71 83.82 0)
+      (effects (font (size 1.27 1.27)) hide)
+    )
     (pin "1")
     (pin "2")
@@
       (effects (font (size 1.27 1.27)) hide)
     )
+    (property "LCSC" "C108661" (id 4) (at 92.71 74.93 0)
+      (effects (font (size 1.27 1.27)) hide)
+    )
     (pin "1")
     (pin "2")
@@
       (effects (font (size 1.27 1.27)) hide)
     )
+    (property "LCSC" "C1713" (id 4) (at 52.07 40.64 0)
+      (effects (font (size 1.27 1.27)) hide)
+    )
